Commit message: urdf addons + realsense r200

File: mockbot/urdf/mockturtlebot.urdf (robot description, URDF)
Before this commit: robot mockturtlebot, 21 links, 20 joints
Links:
- removed link camera_depth_frame
- removed link camera_depth_optical_frame
- removed link camera_link
- removed link camera_rgb_frame
- removed link camera_rgb_optical_frame
- added link r200_link, mass 0.200; collision box size=0.007 0.130 0.02; visual box size=0.007 0.130 0.02
- link back_left_axle: geometry visual cylinder length=0.077 radius=0.01
- link back_left_rim: geometry visual cylinder length=0.075 radius=0.08
- link back_right_axle: geometry visual cylinder length=0.077 radius=0.01
- link back_right_rim: geometry visual cylinder length=0.075 radius=0.08
- link front_left_axle: geometry visual cylinder length=0.077 radius=0.01
- link front_left_rim: geometry visual cylinder length=0.075 radius=0.08
- link front_right_axle: geometry visual cylinder length=0.077 radius=0.01
- link front_right_rim: geometry visual cylinder length=0.075 radius=0.08
Joints:
- removed joint camera_depth_joint
- removed joint camera_depth_optical_joint
- removed joint camera_joint
- removed joint camera_rgb_joint
- removed joint camera_rgb_optical_joint
- added joint r200_joint: type fixed, parent base_link, child r200_link
- joint back_left_rim_joint: origin xyz=-0.15 0.25 0.0 rpy=0 0 0 -> xyz=0 0 0 rpy=0 0 0
- joint back_left_wheel_joint: origin xyz=-0.15 0.25 0.0 rpy=0 0 0 -> xyz=0 0 0 rpy=0 0 0
- joint back_right_rim_joint: origin xyz=-0.15 -0.25 0.0 rpy=0 0 0 -> xyz=0 0 0 rpy=0 0 0
- joint back_right_wheel_joint: origin xyz=-0.15 -0.25 0.0 rpy=0 0 0 -> xyz=0 0 0 rpy=0 0 0
- joint front_left_rim_joint: origin xyz=0.15 0.25 0.0 rpy=0 0 0 -> xyz=0 0 0 rpy=0 0 0
- joint front_left_wheel_joint: origin xyz=0.15 0.25 0.0 rpy=0 0 0 -> xyz=0 0 0 rpy=0 0 0
- joint front_right_rim_joint: origin xyz=0.15 -0.25 0.0 rpy=0 0 0 -> xyz=0 0 0 rpy=0 0 0
- joint front_right_wheel_joint: origin xyz=0.15 -0.25 0.0 rpy=0 0 0 -> xyz=0 0 0 rpy=0 0 0

File: mockbot/urdf/mockturtlebot.urdf.xacro (robot description, xacro)
@@ -5,5 +5,8 @@
   <xacro:include filename="$(find mockbot)/urdf/wheel.urdf.xacro" />
   <xacro:include filename="$(find mockbot)/urdf/addons.urdf.xacro" />
+  <xacro:include filename="$(find mockbot)/urdf/realsense_camera.urdf.xacro" />
+  <!--
   <xacro:include filename="$(find mockbot)/urdf/r200.urdf.xacro" />
+  -->
   <!-- PROPERTY LIST -->
   <!--All units in m-kg-s-radians unit system -->
@@ -45,7 +48,8 @@
   <wheel fb="back" lr="right" parent="base_link" translateX="-1" translateY="-1" flipY="-1"/>
   <wheel fb="back" lr="left" parent="base_link" translateX="-1" translateY="1" flipY="-1"/>
-  <sensor_r200 parent="base_link"/>
+  <realsense_camera_model name="r200" parent="base_link" />
 <!--
   <addonbox xbox="0.1" ybox="0.1" zbox="0.1" parent="base_link"/>
+  <sensor_r200 parent="tower_link"/>
   <sensor_r200 parent="base_link"/>
 -->

File: mockbot/urdf/wheel.urdf.xacro (robot description, xacro)
@@ -4,6 +4,6 @@
   <!-- Wheels definitions -->
   <xacro:property name="wheel_radius" value="0.13" />
-  <xacro:property name="rim_radius" value="0.09" />
-  <xacro:property name="axle_radius" value="0.02" />
+  <xacro:property name="rim_radius" value="0.08" />
+  <xacro:property name="axle_radius" value="0.01" />
   <xacro:property name="wheel_height" value="0.070" />
   <xacro:property name="rim_height" value="0.075" />
@@ -44,8 +44,7 @@
     </link>
     <joint name="${fb}_${lr}_rim_joint" type="fixed">
-      <!-- parent link="${parent}"/-->
       <parent link="${fb}_${lr}_axle"/>
       <child link="${fb}_${lr}_rim"/>
-      <origin xyz="${translateX * base_x_origin_to_wheel_origin} ${translateY * base_y_origin_to_wheel_origin} ${base_z_origin_to_wheel_origin}" rpy="0 0 0" />
+      <origin xyz="0 0 0" rpy="0 0 0" />
       <axis xyz="0 1 0" rpy="0 0 0" />
       <limit effort="100" velocity="100"/>
@@ -63,8 +62,7 @@
     </link>
     <joint name="${fb}_${lr}_wheel_joint" type="fixed">
-      <!-- parent link="${parent}"/-->
       <parent link="${fb}_${lr}_rim"/>
       <child link="${fb}_${lr}_wheel"/>
-      <origin xyz="${translateX * base_x_origin_to_wheel_origin} ${translateY * base_y_origin_to_wheel_origin} ${base_z_origin_to_wheel_origin}" rpy="0 0 0" />
+      <origin xyz="0 0 0" rpy="0 0 0" />
       <axis xyz="0 1 0" rpy="0 0 0" />
       <limit effort="100" velocity="100"/>
